Commit message: refactor env_demo; rename urdf files for stable pushing; add urdf files with fingers

File: gym-bullet-extensions/gym_bullet_extensions/data/yumi_robot/urdf/yumi.urdf (robot description, URDF)
Before this commit: robot yumi, 22 links, 21 joints
Links:
- link gripper_l_finger_l: geometry collision mesh filename=meshes/gripper/coarse/finger.stl; visual mesh filename=meshes/gripper/finger.stl
- link gripper_l_finger_r: geometry collision mesh filename=meshes/gripper/coarse/finger.stl; visual mesh filename=meshes/gripper/finger.stl
- link gripper_r_finger_l: geometry collision mesh filename=meshes/gripper/coarse/finger.stl; visual mesh filename=meshes/gripper/finger.stl
- link gripper_r_finger_r: geometry collision mesh filename=meshes/gripper/coarse/finger.stl; visual mesh filename=meshes/gripper/finger.stl
