Commit message: small urdf correction for Franka full

File: gym-bullet-extensions/gym_bullet_extensions/data/franka_robot/franka_dual.urdf (robot description, URDF)
Before this commit: robot panda, 25 links, 24 joints
Joints:
- joint robot_l_to_world: origin xyz=-0.01 0.83 0.03 rpy=0 0 0 -> xyz=-0.01 -0.83 0.03 rpy=0 0 0

Commit message: update franka full URDF

File: gym-bullet-extensions/gym_bullet_extensions/data/franka_robot/franka_dual.urdf (robot description, URDF)
Before this commit: robot panda, 25 links, 24 joints
Links:
- removed link panda_leftfinger_l
- removed link panda_leftfinger_r
- removed link panda_rightfinger_l
- removed link panda_rightfinger_r
- added link panda_hand_l_finger_l, mass 0.01; collision mesh filename=meshes/collision/finger.stl; visual mesh filename=meshes/visual/finger.dae
- added link panda_hand_l_finger_r, mass 0.01; collision mesh filename=meshes/collision/finger.stl; visual mesh filename=meshes/visual/finger.dae
- added link panda_hand_r_finger_l, mass 0.01; collision mesh filename=meshes/collision/finger.stl; visual mesh filename=meshes/visual/finger.dae
- added link panda_hand_r_finger_r, mass 0.01; collision mesh filename=meshes/collision/finger.stl; visual mesh filename=meshes/visual/finger.dae
Joints:
- removed joint panda_finger_joint1_l
- removed joint panda_finger_joint1_r
- removed joint panda_finger_joint2_l
- removed joint panda_finger_joint2_r
- added joint panda_hand_l_finger_l_joint: type prismatic, parent panda_hand_l, child panda_hand_l_finger_l, origin xyz=0 0 0.0584 rpy=0 0 0, axis 0 1 0, limit lower=0.0 upper=0.04 effort=20 velocity=0.2
- added joint panda_hand_l_finger_r_joint: type prismatic, parent panda_hand_l, child panda_hand_l_finger_r, origin xyz=0 0 0.0584 rpy=0 0 0, axis 0 -1 0, limit lower=0.0 upper=0.04 effort=20 velocity=0.2, mimic joint=panda_hand_l_finger_l_joint
- added joint panda_hand_r_finger_l_joint: type prismatic, parent panda_hand_r, child panda_hand_r_finger_l, origin xyz=0 0 0.0584 rpy=0 0 0, axis 0 1 0, limit lower=0.0 upper=0.04 effort=20 velocity=0.2
- added joint panda_hand_r_finger_r_joint: type prismatic, parent panda_hand_r, child panda_hand_r_finger_r, origin xyz=0 0 0.0584 rpy=0 0 0, axis 0 -1 0, limit lower=0.0 upper=0.04 effort=20 velocity=0.2, mimic joint=panda_hand_r_finger_l_joint
